File: Circuito/Termostato.kicad_sch (KiCad schematic)
At the start: 31 parts

Commit message: Update Termostato.kicad_sch
Parts:
- removed D2: (no value), symbol Device:LED
- removed R5: (no value), symbol Device:R
- BZ1: value (none) -> Buzzer
- C1, C3, C4, C6: value (none) -> 100nf
- C2: value (none) -> 1000uf / 25v
- C7, C9: value (none) -> 100uf
- D1: value (none) -> 1N4001; footprint (none) -> Diode_THT:D_DO-41_SOD81_P10.16mm_Horizontal
- J1: value (none) -> 12v
- J2: value (none) -> Termistor
- J3: value (none) -> ICSP
- J4: value (none) -> 8v
- J5: value (none) -> Peltier
- K1: value (none) -> Relay; footprint (none) -> Relay_THT:Relay_StandexMeder_DIP_LowProfile
- Q1: value (none) -> BC338; footprint (none) -> Package_TO_SOT_THT:TO-92_Inline
- R2, R3: value (none) -> 1K
- R4, R6: value (none) -> 10K
- R7: value (none) -> 33R
- SW1: value (none) -> SUBIR
- SW2: value (none) -> BAJAR
- U1: value (none) -> L78L08_TO92; footprint (none) -> Package_TO_SOT_THT:TO-92_Inline
- U2: value (none) -> L78L05_TO92; footprint (none) -> Package_TO_SOT_THT:TO-92_Inline
- U3: value (none) -> PIC12F675-IP; footprint (none) -> Package_DIP:DIP-8_W7.62mm
Connections:
- net at SW2.3 (K), SW2.4 (A): now also R2.1; no longer R3.1
- net at R3.2, U3.5 (GP2): now also C7.1, R4.1; no longer C3.1
- net at J2.1 (Pin_1): now also R3.1; no longer R1.1
- net at J3.4 (Pin_4), R1.2, U3.7 (GP0): now also C3.1; no longer C7.1, R4.1
- net at SW1.3 (K), SW1.4 (A): now also R1.1; no longer R2.1
